File: nightwing.sch (KiCad schematic (older format))
At the start: 121 parts, among them J1 USB_C_Receptacle_USB2.0, J2 USB_C_Receptacle_USB2.0, J3 OLED, SW1 SW_PUSH, SW10 SW_PUSH, SW11 SW_PUSH, SW12 SW_PUSH, SW13 SW_PUSH, SW14 SW_PUSH, SW15 SW_PUSH, SW16 SW_PUSH, SW17 SW_PUSH, SW18 SW_PUSH, SW19 Rotary_Encoder, SW2 SW_PUSH, SW20 SW_PUSH, SW21 SW_PUSH, SW22 SW_PUSH, SW23 SW_PUSH, SW24 SW_PUSH, SW3 SW_PUSH, SW4 SW_PUSH, SW5 SW_PUSH, SW6 SW_PUSH, SW7 SW_PUSH, SW8 SW_PUSH, SW9 SW_PUSH, U1 ATMEGA32U4, U2 MIC5219-5.0YMM

Commit message: fixed dangling trace a5
Parts:
- 16mhz1: symbol butterfly-rescue:Crystal-Device-monarch-rescue -> nightwing-rescue:Crystal-Device-monarch-rescue-butterfly-rescue
- BZ1: symbol butterfly-rescue:Buzzer-Device-monarch-rescue -> nightwing-rescue:Buzzer-Device-monarch-rescue-butterfly-rescue
- C1: symbol butterfly-rescue:C_Small-Device-monarch-rescue -> nightwing-rescue:C_Small-Device-monarch-rescue-butterfly-rescue
- C19, C6: symbol butterfly-rescue:CP1_Small-Device-monarch-rescue -> nightwing-rescue:CP1_Small-Device-monarch-rescue-butterfly-rescue
- C3, C5, C7, C8: symbol butterfly-rescue:C-Device-monarch-rescue -> nightwing-rescue:C-Device-monarch-rescue-butterfly-rescue
- D1, D10, D11, D12, D13, D14, D15, D16, D17, D18, D19, D2, D20, D21, D22, D23, D24, D25, D3, D4, D5, D6, D7, D8, D9: symbol butterfly-rescue:D-Device-monarch-rescue -> nightwing-rescue:D-Device-monarch-rescue-butterfly-rescue
- D26, D27, RED1: symbol butterfly-rescue:LED-Device-monarch-rescue -> nightwing-rescue:LED-Device-monarch-rescue-butterfly-rescue
- JP1: symbol butterfly-rescue:Jumper-Device-monarch-rescue -> nightwing-rescue:Jumper-Device-monarch-rescue-butterfly-rescue
- R1, R2, R3, R4, R5, R7: symbol butterfly-rescue:R_US-Device-monarch-rescue -> nightwing-rescue:R_US-Device-monarch-rescue-butterfly-rescue
- R6, R8: symbol butterfly-rescue:R_Small_US-Device-monarch-rescue -> nightwing-rescue:R_Small_US-Device-monarch-rescue-butterfly-rescue
- SW19: symbol butterfly-rescue:Rotary_Encoder_Switch-Device-monarch-rescue -> nightwing-rescue:Rotary_Encoder_Switch-Device-monarch-rescue-butterfly-rescue
- U2: symbol butterfly-rescue:MIC5219-5.0YMM-Regulator_Linear-monarch-rescue -> nightwing-rescue:MIC5219-5.0YMM-Regulator_Linear-monarch-rescue-butterfly-rescue
