File: nightwing.sch (KiCad schematic (older format))
At the start: 108 parts, among them J1 USB_C_Receptacle_USB2.0, J2 USB_C_Receptacle_USB2.0, J3 OLED, SW1 SW_PUSH, SW10 SW_PUSH, SW11 SW_PUSH, SW12 SW_PUSH, SW13 SW_PUSH, SW14 SW_PUSH, SW15 SW_PUSH, SW16 SW_PUSH, SW17 SW_PUSH, SW18 SW_PUSH, SW19 Rotary_Encoder, SW2 SW_PUSH, SW20 SW_PUSH, SW21 SW_PUSH, SW22 SW_PUSH, SW23 SW_PUSH, SW24 SW_PUSH, SW3 SW_PUSH, SW4 SW_PUSH, SW5 SW_PUSH, SW6 SW_PUSH, SW7 SW_PUSH, SW8 SW_PUSH, SW9 SW_PUSH, U1 PRTR5V0U2X, U3 ATmega32U4-AU, X1 16mhz

Commit message: updated stm32
Parts:
- removed U?: STM32F103R8Tx, Package_QFP:LQFP-64_10x10mm_P0.5mm, symbol MCU_ST_STM32F1:STM32F103R8Tx
- added L40, L41, L42: WS2812B, reversible-kicad-footprints:ws2812_reversible, symbol LED:WS2812B
Connections:
- wire segments 311 -> 321
- no-connect marks 11 -> 12
Other:
- moved on the sheet: BZ1, L36, L37, L38, L39, X1

Commit message: updated final verseion
Parts:
- added H1, H10, H2, H3, H4, H5, H6, H7, H8, H9: MountingHole, MountingHole:MountingHole_2.2mm_M2_DIN965, symbol Mechanical:MountingHole
- added R1, R6, R8: 5.1k, Resistor_SMD:R_0805_2012Metric, symbol Device:R_Small_US
- renumbered RESET_SW1 to RESET1
Connections:
- net +5V: now also R1.1, R8.1
- net GND: now also R6.2
- net SPLIT_HAND_PIN: now reaches U3.8 (PB0)
- net SPLIT_HAND_PIN: now also R1.2, R6.1
- net PLUG_DETECT: now reaches U3.9 (PB1)
- net PLUG_DETECT: now also R8.2
- no-connect marks 12 -> 10
Other:
- moved on the sheet: BZ1, C1, C10, C2, C4, C5, C9, D1, D10, D11, D12, D13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

Commit message: final output jlcpcb
Parts:
- added BOOT1: SW_PUSH, reversible-kicad-footprints:SW_Push_1P1T_NO_6x6mm_H9.5mm, symbol keyboard_parts:SW_PUSH
Connections:
- net GND: now also BOOT1.2
- net BOOT: now reaches U3.10 (PB2)
- net BOOT: now also BOOT1.1
Changed lines of the file:
@@
 Wire Wire Line
 	6200 1100 6575 1100
-NoConn ~ 8875 1375
 NoConn ~ 8875 1475
 NoConn ~ 8875 1875
@@
 Wire Wire Line
 	9125 1275 8875 1275
+Wire Wire Line
+	2250 3650 2450 3650
+Text GLabel 1650 3650 0    50   Input ~ 0
+BOOT
+$Comp
+L keyboard_parts:SW_PUSH BOOT1
+U 1 1 60CF7BA1
+P 1950 3650
+F 0 "BOOT1" H 1950 3905 50  0000 C CNN
+F 1 "SW_PUSH" H 1950 3814 50  0000 C CNN
+F 2 "reversible-kicad-footprints:SW_Push_1P1T_NO_6x6mm_H9.5mm" H 1950 3650 60  0001 C CNN
+F 3 "" H 1950 3650 60  0000 C CNN
+	1    1950 3650
+	1    0    0    -1
+$EndComp
+$Comp
+L nightwing-rescue:GND-power-monarch-rescue-butterfly-rescue #PWR0111
+U 1 1 60CF7BA7
+P 2450 3650
+F 0 "#PWR0111" H 2450 3400 50  0001 C CNN
+F 1 "GND" V 2450 3450 50  0000 C CNN
+F 2 "" H 2450 3650 50  0001 C CNN
+F 3 "" H 2450 3650 50  0001 C CNN
+	1    2450 3650
+	0    -1   -1   0
+$EndComp
+NoConn ~ 8875 2675
+Text GLabel 9125 1375 2    50   Input ~ 0
+BOOT
+Wire Wire Line
+	9125 1375 8875 1375
 $EndSCHEMATC

Commit message: fixed missing capactior
Parts:
- added C?: 10uf, Capacitor_SMD:C_0805_2012Metric, symbol Device:C_Small
- BOOT1, RESET1, SW1, SW10, SW11, SW12, SW13, SW14, SW15, SW16, SW17, SW18, SW2, SW20, SW21, SW22, SW23, SW24, SW3, SW4, SW5, SW6, SW7, SW8, SW9: symbol keyboard_parts:SW_PUSH -> nightwing-rescue:SW_PUSH-keyboard_parts
- F2: symbol keyboard_parts:PPTC -> nightwing-rescue:PPTC-keyboard_parts
- J1, J2: symbol reversible-kicad-symbols:HRO-TYPE-C-31-M-12-HandSoldering-NoSBU -> nightwing-rescue:HRO-TYPE-C-31-M-12-HandSoldering-NoSBU-reversible-kicad-symbols
- J3: symbol Private:OLED -> nightwing-rescue:OLED-Private
- U1: symbol keebio:PRTR5V0U2X -> nightwing-rescue:PRTR5V0U2X-keebio
- renumbered R1 to LEFT, R6 to RIGHT
Connections:
- net +5V: now also C?.1
- net GND: now also C?.2
Changed lines of the file:
@@
 	2250 1000 2500 1000
 $Comp
-L Private:OLED J3
+L nightwing-rescue:OLED-Private J3
 U 1 1 6061FF7E
 P 1550 4600
@@
 	2250 4050 2450 4050
 $Comp
-L keyboard_parts:SW_PUSH SW24
+L nightwing-rescue:SW_PUSH-keyboard_parts SW24
 U 1 1 6070971B
 P 6700 8175
@@
 $EndComp
 $Comp
-L keyboard_parts:SW_PUSH SW23
+L nightwing-rescue:SW_PUSH-keyboard_parts SW23
 U 1 1 60709715
 P 5700 8175
@@
 $EndComp
 $Comp
-L keyboard_parts:SW_PUSH SW22
+L nightwing-rescue:SW_PUSH-keyboard_parts SW22
 U 1 1 607096FF
 P 4850 8175
@@
 $EndComp
 $Comp
-L keyboard_parts:SW_PUSH SW21
+L nightwing-rescue:SW_PUSH-keyboard_parts SW21
 U 1 1 607096F9
 P 3850 8175
@@
 $EndComp
 $Comp
-L keyboard_parts:SW_PUSH SW20
+L nightwing-rescue:SW_PUSH-keyboard_parts SW20
 U 1 1 607096EC
 P 3000 8175
@@
 $EndComp
 $Comp
-L keyboard_parts:SW_PUSH SW18
+L nightwing-rescue:SW_PUSH-keyboard_parts SW18
 U 1 1 607096C7
 P 6700 7425
@@
 $EndComp
 $Comp
-L keyboard_parts:SW_PUSH SW17
+L nightwing-rescue:SW_PUSH-keyboard_parts SW17
 U 1 1 607096C1
 P 5700 7425
@@
 $EndComp
 $Comp
-L keyboard_parts:SW_PUSH SW16
+L nightwing-rescue:SW_PUSH-keyboard_parts SW16
 U 1 1 607096A9
 P 4850 7425
@@
 $EndComp
 $Comp
-L keyboard_parts:SW_PUSH SW15
+L nightwing-rescue:SW_PUSH-keyboard_parts SW15
 U 1 1 607096A3
 P 3850 7425
@@
 ROW2
 $Comp
-L keyboard_parts:SW_PUSH SW14
+L nightwing-rescue:SW_PUSH-keyboard_parts SW14
 U 1 1 60709693
 P 3000 7425
@@
 $EndComp
 $Comp
-L keyboard_parts:SW_PUSH SW13
+L nightwing-rescue:SW_PUSH-keyboard_parts SW13
 U 1 1 6070968D
 P 2000 7425
@@
 $EndComp
 $Comp
-L keyboard_parts:SW_PUSH SW12
+L nightwing-rescue:SW_PUSH-keyboard_parts SW12
 U 1 1 606ED5B5
 P 6700 6675
@@
 $EndComp
 $Comp
-L keyboard_parts:SW_PUSH SW11
+L nightwing-rescue:SW_PUSH-keyboard_parts SW11
 U 1 1 606ED5AF
 P 5700 6675
@@
 $EndComp
 $Comp
-L keyboard_parts:SW_PUSH SW10
+L nightwing-rescue:SW_PUSH-keyboard_parts SW10
 U 1 1 606ED597
 P 4850 6675
@@
 $EndComp
 $Comp
-L keyboard_parts:SW_PUSH SW9
+L nightwing-rescue:SW_PUSH-keyboard_parts SW9
 U 1 1 606ED591
 P 3850 6675
@@
 $EndComp
 $Comp
-L keyboard_parts:SW_PUSH SW8
+L nightwing-rescue:SW_PUSH-keyboard_parts SW8
 U 1 1 606ED582
 P 3000 6675
@@
 $EndComp
 $Comp
-L keyboard_parts:SW_PUSH SW7
+L nightwing-rescue:SW_PUSH-keyboard_parts SW7
 U 1 1 606ED57C
 P 2000 6675
@@
 COL5
 $Comp
-L keyboard_parts:SW_PUSH SW6
+L nightwing-rescue:SW_PUSH-keyboard_parts SW6
 U 1 1 606C965C
 P 6700 5925
@@
 $EndComp
 $Comp
-L keyboard_parts:SW_PUSH SW5
+L nightwing-rescue:SW_PUSH-keyboard_parts SW5
 U 1 1 606C9656
 P 5700 5925
@@
 	3550 5575 3550 5925
 $Comp
-L keyboard_parts:SW_PUSH SW4
+L nightwing-rescue:SW_PUSH-keyboard_parts SW4
 U 1 1 606C6A7A
 P 4850 5925
@@
 $EndComp
 $Comp
-L keyboard_parts:SW_PUSH SW3
+L nightwing-rescue:SW_PUSH-keyboard_parts SW3
 U 1 1 606C6A74
 P 3850 5925
@@
 RESET
 $Comp
-L keyboard_parts:SW_PUSH RESET1
+L nightwing-rescue:SW_PUSH-keyboard_parts RESET1
 U 1 1 606B5FE8
 P 1950 4050
@@
 $EndComp
 $Comp
-L keyboard_parts:SW_PUSH SW2
+L nightwing-rescue:SW_PUSH-keyboard_parts SW2
 U 1 1 6063E22B
 P 3000 5925
@@
 $EndComp
 $Comp
-L keyboard_parts:SW_PUSH SW1
+L nightwing-rescue:SW_PUSH-keyboard_parts SW1
 U 1 1 6063DEB9
 P 2000 5925
@@
 $EndComp
 $Comp
-L reversible-kicad-symbols:HRO-TYPE-C-31-M-12-HandSoldering-NoSBU J2
+L nightwing-rescue:HRO-TYPE-C-31-M-12-HandSoldering-NoSBU-reversible-kicad-symbols J2
 U 1 1 60658E93
 P 5400 1450
@@
 $EndComp
 $Comp
-L reversible-kicad-symbols:HRO-TYPE-C-31-M-12-HandSoldering-NoSBU J1
+L nightwing-rescue:HRO-TYPE-C-31-M-12-HandSoldering-NoSBU-reversible-kicad-symbols J1
 U 1 1 6056609A
 P 1650 1400
@@
 $EndComp
 $Comp
-L keyboard_parts:PPTC F2
+L nightwing-rescue:PPTC-keyboard_parts F2
 U 1 1 616A3582
 P 3200 800
@@
 	2750 800  2950 800
 $Comp
-L keebio:PRTR5V0U2X U1
+L nightwing-rescue:PRTR5V0U2X-keebio U1
 U 1 1 60D492B4
 P 3150 2650
@@
 $EndComp
 $Comp
-L Device:C_Small C9
-U 1 1 6143C3A3
-P 11875 1450
-F 0 "C9" H 11925 1550 50  0000 L CNN
-F 1 "0.1uf" H 11925 1350 50  0000 L CNN
-F 2 "Capacitor_SMD:C_0805_2012Metric" H 11875 1450 50  0001 C CNN
-F 3 "~" H 11875 1450 50  0001 C CNN
-	1    11875 1450
-	1    0    0    -1
-$EndComp
-$Comp
 L Device:C_Small C5
 U 1 1 6143C399
@@
 $EndComp
 $Comp
-L Device:R_Small_US R1
+L Device:R_Small_US LEFT
 U 1 1 60B0E8DF
 P 5800 3000
-F 0 "R1" H 5868 3046 50  0000 L CNN
+F 0 "LEFT" H 5868 3046 50  0000 L CNN
 F 1 "5.1k" H 5868 2955 50  0000 L CNN
 F 2 "Resistor_SMD:R_0805_2012Metric" H 5800 3000 50  0001 C CNN
@@
 $EndComp
 $Comp
-L Device:R_Small_US R6
+L Device:R_Small_US RIGHT
 U 1 1 60B0F74D
 P 5800 3350
-F 0 "R6" H 5868 3396 50  0000 L CNN
+F 0 "RIGHT" H 5868 3396 50  0000 L CNN
 F 1 "5.1k" H 5868 3305 50  0000 L CNN
 F 2 "Resistor_SMD:R_0805_2012Metric" H 5800 3350 50  0001 C CNN
@@
 BOOT
 $Comp
-L keyboard_parts:SW_PUSH BOOT1
+L nightwing-rescue:SW_PUSH-keyboard_parts BOOT1
 U 1 1 60CF7BA1
 P 1950 3650
@@
 Wire Wire Line
 	9125 1375 8875 1375
+$Comp
+L Device:C_Small C9
+U 1 1 6143C3A3
+P 11875 1450
+F 0 "C9" H 11925 1550 50  0000 L CNN
+F 1 "0.1uf" H 11925 1350 50  0000 L CNN
+F 2 "Capacitor_SMD:C_0805_2012Metric" H 11875 1450 50  0001 C CNN
+F 3 "~" H 11875 1450 50  0001 C CNN
+	1    11875 1450
+	1    0    0    -1
+$EndComp
+$Comp
+L Device:C_Small C?
+U 1 1 60C6B4D7
+P 12225 1450
+F 0 "C?" H 12275 1550 50  0000 L CNN
+F 1 "10uf" H 12275 1350 50  0000 L CNN
+F 2 "Capacitor_SMD:C_0805_2012Metric" H 12225 1450 50  0001 C CNN
+F 3 "~" H 12225 1450 50  0001 C CNN
+	1    12225 1450
+	1    0    0    -1
+$EndComp
+Wire Wire Line
+	11875 1200 12225 1200
+Wire Wire Line
+	12225 1200 12225 1350
+Connection ~ 11875 1200
+Wire Wire Line
+	12225 1550 12225 1700
+Wire Wire Line
+	12225 1700 11875 1700
+Connection ~ 11875 1700
 $EndSCHEMATC
