File: nightwing_curved.kicad_pcb (KiCad board)
At the start: 2 copper layers, 159.6 x 124.2 mm, 109 parts, among them J1 USB_C_Receptacle_USB2.0, J2 USB_C_Receptacle_USB2.0, J3 OLED, SW1 SW_PUSH, SW10 SW_PUSH, SW11 SW_PUSH, SW12 SW_PUSH, SW13 SW_PUSH, SW14 SW_PUSH, SW15 SW_PUSH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

Commit message: final pub
Parts:
- added REF**: MountingHole_2.2mm_M2, MountingHole:MountingHole_2.2mm_M2, F.Cu at (131.5, 82.7)
- added REF**: MountingHole_2.5mm, MountingHole:MountingHole_2.5mm, F.Cu at (192.8, 65.3)
- moved R2 23.6 mm to (141.5, 81.6), turned to 0 degrees
- moved RESET_SW1 18.5 mm to (152.5, 57.0)
- moved C9 17.0 mm to (137.8, 55.9), turned to 0 degrees
- moved C2 15.8 mm to (137.2, 61.9), turned to 0 degrees
- moved C5 12.6 mm to (133.3, 58.9), turned to 0 degrees
- moved C1 9.13 mm to (133.3, 55.9), turned to 0 degrees
- moved C10 8.30 mm to (141.5, 79.3), turned to 0 degrees
- moved L38 8.09 mm to (150.4, 32.0)
- moved L37 4.56 mm to (150.1, 81.1)
- moved C4 3.65 mm to (133.4, 62.5), turned to 0 degrees
- moved J3 2.16 mm to (145.1, 39.2), turned to 15 degrees
- moved J1 1.77 mm to (37.2, 10.2), turned to 180 degrees
Connections:
- J2 pad A4: +5V -> VCC
- J2 pad A7: RX -> Net-(J2-PadA7)
- J2 pad B4: +5V -> VCC
- J2 pad B6: RX -> Net-(J2-PadB6)
- L12 pad 3: GND -> Net-(L12-Pad3)
- U3 pad 1: BUZZER -> Net-(U3-Pad1)
- U3 pad 10: ROT_A -> COL2
- U3 pad 11: ROT_B -> COL3
- U3 pad 12: ROW3 -> Net-(U3-Pad12)
- U3 pad 21: Net-(U3-Pad21) -> ROW0
- U3 pad 22: Net-(U3-Pad22) -> ROW2
- U3 pad 25: Net-(U3-Pad25) -> ROW1
- U3 pad 26: Net-(U3-Pad26) -> ROW3
- U3 pad 28: Net-(U3-Pad28) -> COL4
- U3 pad 29: Net-(U3-Pad29) -> COL5
- U3 pad 30: ROW0 -> Net-(U3-Pad30)
- U3 pad 31: ROW1 -> ROT_A
- U3 pad 32: ROW2 -> ROT_B
- U3 pad 38: COL5 -> BUZZER
- U3 pad 39: COL4 -> Net-(U3-Pad39)
- U3 pad 40: COL3 -> Net-(U3-Pad40)
- U3 pad 41: COL2 -> Net-(U3-Pad41)
- U3 pad 8: COL1 -> COL0
- U3 pad 9: COL0 -> COL1
Routing:
- net +5V: track 983.4 -> 728.8 mm, vias 38 -> 16
- net SK_LED: track 182.8 -> 0.00 mm, vias 2 -> 0
- net GND: track 143.7 -> 42.3 mm, vias 21 -> 4
- net ROW1: track 180.1 -> 119.0 mm, vias 2 -> 0
- net WS_LED: track 61.5 -> 3.21 mm, vias 3 -> 1
- net Net-(L37-Pad2): track 57.5 -> 0.00 mm, vias 3 -> 0
- net RESET: track 57.1 -> 0.00 mm, vias 4 -> 0
- net SCL: track 56.6 -> 0.00 mm, vias 1 -> 0
- net SDA: track 50.7 -> 0.00 mm, vias 1 -> 0
- net ROW0: track 204.0 -> 158.5 mm, vias 2 -> 1
- net Net-(L38-Pad2): track 33.3 -> 0.00 mm, vias 2 -> 0
- net ROW3: track 133.0 -> 101.1 mm, vias 1 -> 0
- net RX: track 44.6 -> 14.8 mm, vias 2 -> 1
- net ROW2: track 167.3 -> 138.2 mm, vias 0 -> 1
- net COL5: track 130.3 -> 106.7 mm, vias 4 -> 3
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Other:
- board size 159.6 x 124.2 mm -> 177.3 x 129.6 mm
- board text added: "nightwing rev1.0"
