File: stm_nightwing/nightwing.kicad_pcb (KiCad board)
At the start: 2 copper layers, 165.4 x 129.6 mm, 109 parts, among them J1 USB_C_Receptacle_USB2.0, J2 USB_C_Receptacle_USB2.0, J3 OLED, SW1 SW_PUSH, SW10 SW_PUSH, SW11 SW_PUSH, SW12 SW_PUSH, SW13 SW_PUSH, SW14 SW_PUSH, SW15 SW_PUSH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

Commit message: stm_nightwing finished
Parts:
- removed C1, C2, C4, C5, C9: 0.1uf, Capacitor_SMD:C_0805_2012Metric
- removed C10: 1u, Capacitor_SMD:C_0805_2012Metric
- removed RESET_SW1: SW_PUSH, reversible-kicad-footprints:SW_Push_1P1T_NO_6x6mm_H9.5mm
- removed U3: ATmega32U4-AU, Package_QFP:TQFP-44_10x10mm_P0.8mm
- added BOOT: BOOT0, reversible-kicad-footprints:SW_Push_1P1T_NO_6x6mm_H9.5mm, F.Cu at (139.4, 90.7)
- added C11: 100nf, Capacitor_SMD:C_0805_2012Metric_Pad1.18x1.45mm_HandSolder, F.Cu at (136.7, 72.4)
- added C12: 100nf, Capacitor_SMD:C_0805_2012Metric_Pad1.18x1.45mm_HandSolder, F.Cu at (161.0, 72.3)
- added C13: 100nf, Capacitor_SMD:C_0805_2012Metric_Pad1.18x1.45mm_HandSolder, F.Cu at (150.0, 64.0)
- added C14: 100nf, Capacitor_SMD:C_0805_2012Metric_Pad1.18x1.45mm_HandSolder, F.Cu at (161.0, 74.4)
- added C15: 100nf, Capacitor_SMD:C_0805_2012Metric_Pad1.18x1.45mm_HandSolder, F.Cu at (146.0, 64.0)
- added C16: 100nf, Capacitor_SMD:C_0805_2012Metric_Pad1.18x1.45mm_HandSolder, F.Cu at (133.3, 87.0)
- added C17: 0.1uf, Capacitor_SMD:C_0805_2012Metric_Pad1.18x1.45mm_HandSolder, F.Cu at (146.1, 56.4)
- added C18: 0.1uf, Capacitor_SMD:C_0805_2012Metric_Pad1.18x1.45mm_HandSolder, F.Cu at (143.1, 56.3)
- added C3: 10uf, Capacitor_SMD:C_0805_2012Metric_Pad1.18x1.45mm_HandSolder, F.Cu at (159.4, 63.3)
- added C6: 100nf, Capacitor_SMD:C_0805_2012Metric_Pad1.18x1.45mm_HandSolder, F.Cu at (136.7, 74.5)
- added C7: 100nf, Capacitor_SMD:C_0805_2012Metric_Pad1.18x1.45mm_HandSolder, F.Cu at (148.6, 84.2)
- added C8: 100nf, Capacitor_SMD:C_0805_2012Metric_Pad1.18x1.45mm_HandSolder, F.Cu at (146.6, 84.2)
- added F1: PPTC 1.5A, Fuse:Fuse_1206_3216Metric, F.Cu at (163.7, 112.0)
- added G***: LOGO, private:icon_nightwing, F.Cu at (0.04, 40.5)
- added G***: LOGO, private:tiny_nightwing, F.Cu at (37.1, 38.7)
- added G***: LOGO, private:icon_nightwing, F.Cu at (152.8, 90.2)
- added H1: MountingHole, MountingHole:MountingHole_2.2mm_M2_DIN965, F.Cu at (38.5, 62.5)
- added H2: MountingHole, MountingHole:MountingHole_2.2mm_M2_DIN965, F.Cu at (39.0, 81.7)
- added H3: MountingHole, MountingHole:MountingHole_2.2mm_M2_DIN965, F.Cu at (77.0, 44.2)
- added H4: MountingHole, MountingHole:MountingHole_2.2mm_M2_DIN965, F.Cu at (80.2, 83.0)
- added H5: MountingHole, MountingHole:MountingHole_2.2mm_M2_DIN965, F.Cu at (113.5, 54.4)
- added H6: MountingHole, MountingHole:MountingHole_2.2mm_M2_DIN965, F.Cu at (120.2, 94.6)
- added H7: MountingHole, MountingHole:MountingHole_2.2mm_M2_DIN965, F.Cu at (163.5, 105.0)
- added H8: MountingHole, MountingHole:MountingHole_2.2mm_M2_DIN965, F.Cu at (157.8, 135.5)
- added L40: WS2812B, reversible-kicad-footprints:ws2812_reversible, B.Cu at (86.9, 87.1)
- added L41: WS2812B, reversible-kicad-footprints:ws2812_reversible, B.Cu at (101.2, 30.7)
- added L42: WS2812B, reversible-kicad-footprints:ws2812_reversible, B.Cu at (66.2, 25.0)
- added R1: 10k, Resistor_SMD:R_0805_2012Metric, F.Cu at (133.3, 83.4)
- added R10: 9.1k, Resistor_SMD:R_0805_2012Metric, F.Cu at (173.0, 113.7)
- added R11: 9.1k, Resistor_SMD:R_0805_2012Metric, F.Cu at (171.0, 113.4)
- added R12: 68k, Resistor_SMD:R_0805_2012Metric, F.Cu at (139.5, 50.2)
- added R13: 68k, Resistor_SMD:R_0805_2012Metric, F.Cu at (139.5, 53.7)
- added R14: 68k, Resistor_SMD:R_0805_2012Metric, F.Cu at (139.5, 57.2)
- added R6: 9.1k (Left), Resistor_SMD:R_0805_2012Metric, F.Cu at (157.6, 67.4)
- added R8: 9.1k (Right), Resistor_SMD:R_0805_2012Metric, F.Cu at (155.6, 67.4)
- added R9: 9.1k, Resistor_SMD:R_0805_2012Metric, F.Cu at (167.1, 112.7)
- added RESET: RESET, reversible-kicad-footprints:SW_Push_1P1T_NO_6x6mm_H9.5mm, F.Cu at (139.4, 83.7)
- added U2: AP2204RB-3.3, Package_TO_SOT_SMD:SOT-89-3, F.Cu at (144.6, 51.8)
- added U4: STM32F103R8Tx, Package_QFP:LQFP-64_10x10mm_P0.5mm, F.Cu at (148.0, 73.4)
- F2: value PPTC -> PPTC 3A
- J2: moved to F.Cu
- R2: value 10k -> 9.1k
- moved R2 54.8 mm to (169.1, 113.0), turned to 80 degrees
- moved L37 17.6 mm to (150.0, 103.2)
- moved J2 12.8 mm to (171.8, 105.4), turned to 170 degrees
- moved U1 12.4 mm to (28.5, 26.8), turned to 180 degrees
- moved D23 11.7 mm to (136.7, 112.8)
- moved L16 11.7 mm to (85.5, 66.9)
- moved L17 11.7 mm to (104.5, 76.9)
- moved L18 11.7 mm to (123.5, 78.9)
- moved SW12 11.7 mm to (123.5, 65.4)
- moved SW16 11.7 mm to (85.5, 72.4)
- moved SW17 11.7 mm to (104.5, 82.4)
- moved SW18 11.7 mm to (123.5, 84.4)
- moved D13 11.7 mm to (21.9, 86.2)
- moved D14 11.7 mm to (39.3, 87.4)
- moved D15 11.7 mm to (58.3, 71.9)
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Connections:
- J2 pad A4: +5V -> Net-(F1-Pad1)
- J2 pad A6: RX -> SPLIT_COMMS+
- J2 pad A7: RX -> SPLIT_COMMS-
- J2 pad B4: +5V -> Net-(F1-Pad1)
- J2 pad B6: RX -> SPLIT_COMMS+
- J2 pad B7: RX -> SPLIT_COMMS-
- L36 pad 4: Net-(L35-Pad2) -> Net-(L36-Pad4)
- R2 pad 1: GND -> +3V3
- R2 pad 2: Net-(R2-Pad2) -> SPLIT_COMMS-
- X1 pad 1: XTAL1 -> OSC_IN
- X1 pad 2: XTAL2 -> OSC_OUT
Routing:
- net +3V3: track 0.00 -> 169.2 mm, vias 0 -> 7
- net Net-(L36-Pad4): track 0.00 -> 79.9 mm, vias 0 -> 3
- net SPLIT_COMMS+: track 0.00 -> 74.8 mm, vias 0 -> 3
- net SPLIT_COMMS-: track 0.00 -> 69.9 mm, vias 0 -> 4
- net RESET: track 57.1 -> 0.00 mm, vias 4 -> 0
- net RX: track 44.6 -> 0.00 mm, vias 2 -> 0
- net Net-(L41-Pad2): track 0.00 -> 41.3 mm, vias 0 -> 3
- net +5V: track 983.4 -> 943.1 mm, vias 38 -> 32
- net Net-(L35-Pad2): track 78.2 -> 43.9 mm, vias 2 -> 3
- net Net-(L39-Pad2): track 3.85 -> 36.8 mm, vias 1 -> 2
- net ROW0: track 204.0 -> 172.9 mm
- net NRST: track 0.00 -> 27.7 mm, vias 0 -> 4
- net ROW1: track 180.1 -> 153.5 mm, vias 2 -> 0
- net ROW3: track 133.0 -> 158.8 mm, vias 1 -> 2
- net DN: track 183.3 -> 159.8 mm, vias 5 -> 4
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Other:
- board size 165.4 x 129.6 mm -> 158.2 x 125.4 mm
- board text added: "Nightwing v1.0"

Commit message: updated stm32
Parts:
- removed the G*** at (0.04, 40.5)
- C17, C18: value 0.1uf -> 100nf
- moved C12 1.22 mm to (160.3, 71.3)
- moved C14 1.22 mm to (160.3, 73.4)
- renumbered RESET to SW25, BOOT to SW26
Routing:
- net SDA: track 53.9 -> 56.3 mm
- net +3V3: track 169.2 -> 166.9 mm
- net SCL: track 55.1 -> 57.3 mm
