File: stm_nightwing/nightwing.sch (KiCad schematic (older format))
At the start: 124 parts, among them J1 USB_C_Receptacle_USB2.0, J2 USB_C_Receptacle_USB2.0, J3 OLED, SW1 SW_PUSH, SW10 SW_PUSH, SW11 SW_PUSH, SW12 SW_PUSH, SW13 SW_PUSH, SW14 SW_PUSH, SW15 SW_PUSH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

Commit message: stm_nightwing finished
Parts:
- removed C1, C2, C4, C5, C9: 0.1uf, Capacitor_SMD:C_0805_2012Metric, symbol Device:C_Small
- removed C10: 1u, Capacitor_SMD:C_0805_2012Metric, symbol Device:C_Small
- removed R2: 10k, Resistor_SMD:R_0805_2012Metric, symbol Device:R_Small
- removed RESET_SW1: SW_PUSH, reversible-kicad-footprints:SW_Push_1P1T_NO_6x6mm_H9.5mm, symbol keyboard_parts:SW_PUSH
- removed U3: ATmega32U4-AU, Package_QFP:TQFP-44_10x10mm_P0.8mm, symbol MCU_Microchip_ATmega:ATmega32U4-AU
- added F1: PPTC 1.5A, Fuse:Fuse_1206_3216Metric, symbol keyboard_parts:PPTC
- added H1, H2, H3, H4, H5, H6, H7, H8: MountingHole, MountingHole:MountingHole_2.2mm_M2_DIN965, symbol Mechanical:MountingHole
- added L40, L41, L42: WS2812B, reversible-kicad-footprints:ws2812_reversible, symbol LED:WS2812B
- added R10, R11, R2, R9: 9.1k, Resistor_SMD:R_0805_2012Metric, symbol Device:R_Small_US
- added R12, R13, R14: 68k, Resistor_SMD:R_0805_2012Metric, symbol Device:R_Small_US
- added R6: 9.1k (Left), Resistor_SMD:R_0805_2012Metric, symbol Device:R_Small_US
- added R8: 9.1k (Right), Resistor_SMD:R_0805_2012Metric, symbol Device:R_Small_US
- C11, C12, C13, C14, C15, C16, C17, C18, C3, C6, C7, C8: renamed from C?; footprint (none) -> Capacitor_SMD:C_0805_2012Metric_Pad1.18x1.45mm_HandSolder
- F2: value PPTC -> PPTC 3A
- R1: renamed from R?; footprint (none) -> Resistor_SMD:R_0805_2012Metric
- SW26: renamed from SW?; footprint (none) -> reversible-kicad-footprints:SW_Push_1P1T_NO_6x6mm_H9.5mm
- gave numbers to parts that had none: 3
Connections:
- net XTAL1 is gone; now on net OSC_IN: X1.1
- net XTAL2 is gone; now on net OSC_OUT: X1.2
- net +3V3: now also R10.1, R11.1, R2.1, R6.1, R9.1
- net +5V: now also F1.2, L40.1 (VDD), L41.1 (VDD), L42.1 (VDD), R12.1; no longer J2.A4 (VBUS), J2.B4 (VBUS)
- net BUZZER: now also U4.53 (PC12)
- net COL0: now also U4.56 (PB4)
- net COL1: now also U4.55 (PB3)
- net COL2: now also U4.52 (PC11)
- net COL3: now also U4.51 (PC10)
- net COL4: now also U4.50 (PA15)
- net COL5: now also U4.49 (PA14)
- net GND: now also L40.3 (VSS), L41.3 (VSS), L42.3 (VSS), R14.2, R8.2
- net ROT_A: now also U4.61 (PB8)
- net ROT_B: now also U4.62 (PB9)
- net ROW0: now also U4.40 (PC9)
- net ROW1: now also U4.41 (PA8)
- net ROW2: now also U4.42 (PA9)
- net ROW3: now also U4.43 (PA10)
- net SCL: now also U4.58 (PB6); no longer U4.29 (PB10)
- net SDA: now also U4.59 (PB7); no longer U4.30 (PB11)
- net SK_LED: now also U4.39 (PC8)
- net WS_LED: now also U4.38 (PC7)
- net SPLIT_HAND_PIN: now reaches U4.28 (PB2)
- net SPLIT_HAND_PIN: now also R6.2, R8.1
- net PLUG_DETECT: now reaches U4.37 (PC6)
- net PLUG_DETECT: now also R12.2, R13.1
- net OSC_IN: now reaches U4.5 (PD0)
- net OSC_OUT: now reaches U4.6 (PD1)
- net at L36.4 (DIN): now also L40.2 (DOUT); no longer L35.2 (DOUT)
- net at L39.2 (DOUT): now also L41.4 (DIN)
- net RX renamed SPLIT_COMMS+
- net SPLIT_COMMS+: now also U4.30 (PB11), R10.2, R11.2; no longer J2.A7 (D-), J2.B7 (D-)
- new net: F1.1, J2.A4 (VBUS), J2.B4 (VBUS)
- new net: R13.2, R14.1
- new net: L41.2 (DOUT), L42.4 (DIN)
- new net: L35.2 (DOUT), L40.4 (DIN)
- new net SPLIT_COMMS-: J2.A7 (D-), J2.B7 (D-), R2.2, R9.2, U4.29 (PB10)
- no-connect marks 11 -> 3
Other:
- note added: "Left=High\nRight=Low"
- moved on the sheet: C11, C12, C13, C14, C15, C16, C17, C18, C3, C6, C7, C8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

Commit message: updated stm32
Parts:
- C17, C18: value 0.1uf -> 100nf
Other:
- moved on the sheet: BZ1, U1, X1
Changed lines of the file:
@@
 ROW0
-Wire Wire Line
-	1650 1375 1850 1375
-Wire Wire Line
-	1650 1575 1850 1575
 Wire Wire Line
 	2150 1125 2350 1125
@@
 L nightwing-rescue:Crystal-Device-monarch-rescue-butterfly-rescue X1
 U 1 1 612C758C
-P 14450 2950
-F 0 "X1" V 14400 2500 50  0000 L CNN
-F 1 "16mhz" V 14500 2500 50  0000 L CNN
-F 2 "Crystal:Crystal_HC49-4H_Vertical" H 14450 2950 50  0001 C CNN
-F 3 "~" H 14450 2950 50  0001 C CNN
-	1    14450 2950
+P 9550 4700
+F 0 "X1" V 9500 4250 50  0000 L CNN
+F 1 "16mhz" V 9600 4250 50  0000 L CNN
+F 2 "Crystal:Crystal_HC49-4H_Vertical" H 9550 4700 50  0001 C CNN
+F 3 "~" H 9550 4700 50  0001 C CNN
+	1    9550 4700
 	0    1    1    0
 $EndComp
-Text GLabel 13850 2750 0    50   Input ~ 0
+Text GLabel 8950 4500 0    50   Input ~ 0
 OSC_IN
-Text GLabel 13850 3150 0    50   Input ~ 0
+Text GLabel 8950 4900 0    50   Input ~ 0
 OSC_OUT
 Wire Wire Line
-	13850 3150 14450 3150
-Wire Wire Line
-	14450 3150 14450 3100
-Wire Wire Line
-	14450 2800 14450 2750
-Wire Wire Line
-	14450 2750 13850 2750
+	8950 4900 9550 4900
+Wire Wire Line
+	9550 4900 9550 4850
+Wire Wire Line
+	9550 4550 9550 4500
+Wire Wire Line
+	9550 4500 8950 4500
 $Comp
 L power:VCC #PWR02
@@
 L nightwing-rescue:Buzzer-Device-monarch-rescue-butterfly-rescue BZ1
 U 1 1 606C87A5
-P 14050 2450
-F 0 "BZ1" V 14300 2350 50  0000 L CNN
-F 1 "Buzzer" V 14200 2300 50  0000 L CNN
-F 2 "private:Buzzer" V 14025 2550 50  0001 C CNN
-F 3 "~" V 14025 2550 50  0001 C CNN
-	1    14050 2450
+P 9150 4200
+F 0 "BZ1" V 9400 4100 50  0000 L CNN
+F 1 "Buzzer" V 9300 4050 50  0000 L CNN
+F 2 "private:Buzzer" V 9125 4300 50  0001 C CNN
+F 3 "~" V 9125 4300 50  0001 C CNN
+	1    9150 4200
 	0    -1   -1   0
 $EndComp
-Text GLabel 13800 2550 0    50   Input ~ 0
+Text GLabel 8900 4300 0    50   Input ~ 0
 BUZZER
 Wire Wire Line
-	13950 2550 13800 2550
+	9050 4300 8900 4300
 $Comp
 L power:GND #PWR07
 U 1 1 61DDD2A6
-P 14300 2550
-F 0 "#PWR07" H 14300 2300 50  0001 C CNN
-F 1 "GND" V 14305 2422 50  0000 R CNN
-F 2 "" H 14300 2550 50  0001 C CNN
-F 3 "" H 14300 2550 50  0001 C CNN
-	1    14300 2550
+P 9400 4300
+F 0 "#PWR07" H 9400 4050 50  0001 C CNN
+F 1 "GND" V 9405 4172 50  0000 R CNN
+F 2 "" H 9400 4300 50  0001 C CNN
+F 3 "" H 9400 4300 50  0001 C CNN
+	1    9400 4300
 	0    -1   -1   0
 $EndComp
 Wire Wire Line
-	14150 2550 14300 2550
+	9250 4300 9400 4300
 Connection ~ 14700 8550
 Connection ~ 14700 7150
@@
 	0    1    1    0
 $EndComp
-Text GLabel 2350 1375 2    50   Input ~ 0
-D-
-Text GLabel 2350 1575 2    50   Input ~ 0
-D+
-$Comp
-L nightwing-rescue:R_US-Device-monarch-rescue-butterfly-rescue R5
-U 1 1 608DE27F
-P 2000 1375
-F 0 "R5" V 1950 1225 50  0000 C CNN
-F 1 "22" V 1950 1525 50  0000 C CNN
-F 2 "Resistor_SMD:R_0805_2012Metric" V 2040 1365 50  0001 C CNN
-F 3 "~" H 2000 1375 50  0001 C CNN
-	1    2000 1375
-	0    1    1    0
-$EndComp
-$Comp
-L nightwing-rescue:R_US-Device-monarch-rescue-butterfly-rescue R7
-U 1 1 60900530
-P 2000 1575
-F 0 "R7" V 1950 1425 50  0000 C CNN
-F 1 "22" V 1950 1725 50  0000 C CNN
-F 2 "Resistor_SMD:R_0805_2012Metric" V 2040 1565 50  0001 C CNN
-F 3 "~" H 2000 1575 50  0001 C CNN
-	1    2000 1575
-	0    1    1    0
-$EndComp
-Wire Wire Line
-	2150 1375 2350 1375
-Wire Wire Line
-	2150 1575 2350 1575
 Wire Wire Line
 	1650 1325 1650 1375
@@
 Text Notes 3725 4750 0    50   ~ 0
 Left=High\nRight=Low
-Text GLabel 12900 4325 2    50   Input ~ 0
-SPLIT_COMMS+
-Text GLabel 12900 4225 2    50   Input ~ 0
-SPLIT_COMMS-
-Wire Wire Line
-	12900 4325 12675 4325
-Wire Wire Line
-	12675 4225 12900 4225
 Wire Wire Line
 	8250 1925 8050 1925
@@
 Text GLabel 12875 4025 2    50   Input ~ 0
 ROT_A
-Text GLabel 11075 4425 0    50   Input ~ 0
-BUZZER
 Text GLabel 12875 2525 2    50   Input ~ 0
 ROW3
@@
 Text GLabel 12875 2325 2    50   Input ~ 0
 ROW1
-Text GLabel 11075 4125 0    50   Input ~ 0
-ROW0
 Text GLabel 12875 3625 2    50   Input ~ 0
 COL0
@@
 Text GLabel 12875 3025 2    50   Input ~ 0
 COL4
-Text GLabel 11075 4225 0    50   Input ~ 0
-COL3
-Text GLabel 11075 4325 0    50   Input ~ 0
-COL2
 Text GLabel 12875 3525 2    50   Input ~ 0
 COL1
-Text GLabel 11075 3925 0    50   Input ~ 0
-WS_LED
-Text GLabel 11075 4025 0    50   Input ~ 0
-SK_LED
 Wire Wire Line
 	12875 3625 12675 3625
@@
 	12675 3525 12875 3525
 Wire Wire Line
-	11075 4325 11275 4325
-Wire Wire Line
-	11275 4225 11075 4225
-Wire Wire Line
 	12875 3025 12675 3025
 Wire Wire Line
 	12675 2925 12875 2925
 Wire Wire Line
-	11075 4025 11275 4025
-Wire Wire Line
-	11275 3925 11075 3925
-Wire Wire Line
-	11075 4125 11275 4125
-Wire Wire Line
 	12675 2325 12875 2325
 Wire Wire Line
@@
 	12675 2525 12875 2525
 Wire Wire Line
-	11275 4425 11075 4425
-Wire Wire Line
 	12875 4025 12675 4025
-Wire Wire Line
-	12675 4125 12875 4125
 Wire Wire Line
 	8050 2025 8050 1925
@@
 	1    0    0    -1
 $EndComp
-Text GLabel 11075 3825 0    50   Input ~ 0
-PLUG_DETECT
-Wire Wire Line
-	11275 3825 11075 3825
 $Comp
 L power:+5V #PWR03
@@
 P 2075 4000
 F 0 "C18" H 2167 4046 50  0000 L CNN
-F 1 "0.1uf" H 2167 3955 50  0000 L CNN
+F 1 "100nf" H 2167 3955 50  0000 L CNN
 F 2 "Capacitor_SMD:C_0805_2012Metric_Pad1.18x1.45mm_HandSolder" H 2075 4000 50  0001 C CNN
 F 3 "~" H 2075 4000 50  0001 C CNN
@@
 P 1050 4000
 F 0 "C17" H 1142 4046 50  0000 L CNN
-F 1 "0.1uf" H 1142 3955 50  0000 L CNN
+F 1 "100nf" H 1142 3955 50  0000 L CNN
 F 2 "Capacitor_SMD:C_0805_2012Metric_Pad1.18x1.45mm_HandSolder" H 1050 4000 50  0001 C CNN
 F 3 "~" H 1050 4000 50  0001 C CNN
@@
 	1    0    0    -1
 $EndComp
+Text GLabel 1900 2375 0    50   Input ~ 0
+DN
+Wire Wire Line
+	1650 1575 1850 1575
+Wire Wire Line
+	1650 1375 1850 1375
+Wire Wire Line
+	2150 1575 2350 1575
+Wire Wire Line
+	2150 1375 2350 1375
+Text GLabel 2350 1575 2    50   Input ~ 0
+D+
+Text GLabel 2350 1375 2    50   Input ~ 0
+D-
+$Comp
+L nightwing-rescue:R_US-Device-monarch-rescue-butterfly-rescue R7
+U 1 1 60900530
+P 2000 1575
+F 0 "R7" V 1950 1425 50  0000 C CNN
+F 1 "22" V 1950 1725 50  0000 C CNN
+F 2 "Resistor_SMD:R_0805_2012Metric" V 2040 1565 50  0001 C CNN
+F 3 "~" H 2000 1575 50  0001 C CNN
+	1    2000 1575
+	0    1    1    0
+$EndComp
+$Comp
+L nightwing-rescue:R_US-Device-monarch-rescue-butterfly-rescue R5
+U 1 1 608DE27F
+P 2000 1375
+F 0 "R5" V 1950 1225 50  0000 C CNN
+F 1 "22" V 1950 1525 50  0000 C CNN
+F 2 "Resistor_SMD:R_0805_2012Metric" V 2040 1365 50  0001 C CNN
+F 3 "~" H 2000 1375 50  0001 C CNN
+	1    2000 1375
+	0    1    1    0
+$EndComp
+$Comp
+L power:GND #PWR08
+U 1 1 60D51B38
+P 1900 2275
+F 0 "#PWR08" H 1900 2025 50  0001 C CNN
+F 1 "GND" V 1905 2147 50  0000 R CNN
+F 2 "" H 1900 2275 50  0001 C CNN
+F 3 "" H 1900 2275 50  0001 C CNN
+	1    1900 2275
+	0    1    1    0
+$EndComp
+$Comp
+L power:VCC #PWR09
+U 1 1 60D51023
+P 2600 2275
+F 0 "#PWR09" H 2600 2125 50  0001 C CNN
+F 1 "VCC" V 2615 2403 50  0000 L CNN
+F 2 "" H 2600 2275 50  0001 C CNN
+F 3 "" H 2600 2275 50  0001 C CNN
+	1    2600 2275
+	0    1    1    0
+$EndComp
+Text GLabel 2600 2375 2    50   Input ~ 0
+DP
 $Comp
 L keebio:PRTR5V0U2X U1
 U 1 1 60D492B4
-P 1175 3050
-F 0 "U1" H 1175 3325 50  0000 C CNN
-F 1 "PRTR5V0U2X" H 1175 3234 50  0000 C CNN
-F 2 "Package_TO_SOT_SMD:SOT-143_Handsoldering" H 1125 3150 50  0001 C CNN
-F 3 "" H 1125 3150 50  0001 C CNN
-	1    1175 3050
-	1    0    0    -1
-$EndComp
-Text GLabel 825  3100 0    50   Input ~ 0
-DN
-Text GLabel 1525 3100 2    50   Input ~ 0
-DP
-$Comp
-L power:VCC #PWR09
-U 1 1 60D51023
-P 1525 3000
-F 0 "#PWR09" H 1525 2850 50  0001 C CNN
-F 1 "VCC" V 1540 3128 50  0000 L CNN
-F 2 "" H 1525 3000 50  0001 C CNN
-F 3 "" H 1525 3000 50  0001 C CNN
-	1    1525 3000
-	0    1    1    0
-$EndComp
-$Comp
-L power:GND #PWR08
-U 1 1 60D51B38
-P 825 3000
-F 0 "#PWR08" H 825 2750 50  0001 C CNN
-F 1 "GND" V 830 2872 50  0000 R CNN
-F 2 "" H 825 3000 50  0001 C CNN
-F 3 "" H 825 3000 50  0001 C CNN
-	1    825  3000
-	0    1    1    0
-$EndComp
+P 2250 2325
+F 0 "U1" H 2250 2600 50  0000 C CNN
+F 1 "PRTR5V0U2X" H 2250 2509 50  0000 C CNN
+F 2 "Package_TO_SOT_SMD:SOT-143_Handsoldering" H 2200 2425 50  0001 C CNN
+F 3 "" H 2200 2425 50  0001 C CNN
+	1    2250 2325
+	1    0    0    -1
+$EndComp
+Text GLabel 12900 4225 2    50   Input ~ 0
+SPLIT_COMMS-
+Text GLabel 12900 4325 2    50   Input ~ 0
+SPLIT_COMMS+
+Wire Wire Line
+	12900 4325 12675 4325
+Wire Wire Line
+	12675 4225 12900 4225
+Wire Wire Line
+	12675 4125 12875 4125
+Wire Wire Line
+	11275 3825 11075 3825
+Text GLabel 11075 3825 0    50   Input ~ 0
+PLUG_DETECT
+Wire Wire Line
+	11275 4425 11075 4425
+Wire Wire Line
+	11075 4125 11275 4125
+Wire Wire Line
+	11275 3925 11075 3925
+Wire Wire Line
+	11075 4025 11275 4025
+Wire Wire Line
+	11275 4225 11075 4225
+Wire Wire Line
+	11075 4325 11275 4325
+Text GLabel 11075 4025 0    50   Input ~ 0
+SK_LED
+Text GLabel 11075 3925 0    50   Input ~ 0
+WS_LED
+Text GLabel 11075 4325 0    50   Input ~ 0
+COL2
+Text GLabel 11075 4225 0    50   Input ~ 0
+COL3
+Text GLabel 11075 4125 0    50   Input ~ 0
+ROW0
+Text GLabel 11075 4425 0    50   Input ~ 0
+BUZZER
 $EndSCHEMATC
